File: abqmmf2018.brd (EAGLE design)
At the start: 125.5 x 93.7 mm, 13 parts

Commit message: Remove accidental double reference
S2, Pad 3 was accidentally assigned to both GPIO15 and GPIO5/SCL
Removing GPIO15 since 5 is what's actually routed
Connections:
- net GPIO15: no longer S2.3
Changed lines of the file:
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@@
 <signal name="GPIO15">
 <contactref element="AMICA-NODEMCU" pad="D8"/>
-<contactref element="S2" pad="3"/>
 <contactref element="JP2" pad="14"/>
 <wire x1="100.33" y1="27.94" x2="100.33" y2="10.16" width="0" layer="19" extent="1-16"/>

Commit message: Removing Buttons for GPIO9/10
These are basically unusable on a certain portion of NodeMCUs,
so removing them entirely
Parts:
- removed S4, S5: MOMENTARY-SWITCH-SPST-PTH-6.0MM, SparkFun-Switches:TACTILE_SWITCH_PTH_6.0MM
Connections:
- net GND: no longer S4.1, S5.1
- net GPIO10: no longer S5.3
- net GPIO9: no longer S4.3
Routing:
- net GPIO9: track 112.5 -> 65.0 mm, vias 1 -> 0
- net GPIO10: track 90.5 -> 83.5 mm
Other:
- board text removed: "GPIO10"
- board text removed: "GPIO9"
Changed lines of the file:
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@@
 <text x="40.64" y="29.21" size="1.27" layer="22" font="vector" rot="MR90">Reminder: put the battery holder on last!</text>
 <text x="51.7525" y="26.3525" size="1.27" layer="21" font="vector" rot="R270">GPIO13</text>
-<text x="41.275" y="16.51" size="1.27" layer="21" font="vector" rot="R270">GPIO9</text>
 <text x="51.435" y="17.4625" size="1.27" layer="21" font="vector" rot="R270">GPIO12</text>
-<text x="61.595" y="17.4625" size="1.27" layer="21" font="vector" rot="R270">GPIO10</text>
 <text x="51.435" y="8.89" size="1.27" layer="21" font="vector" rot="R270">GPIO15</text>
 <text x="65.405" y="73.3425" size="0.8128" layer="21" font="vector" rot="R45">TXD</text>
@@
 <attribute name="NAME" x="46.99" y="19.558" size="0.6096" layer="25" font="vector" ratio="20" rot="R180" align="bottom-center"/>
 </element>
-<element name="S4" library="SparkFun-Switches" package="TACTILE_SWITCH_PTH_6.0MM" value="MOMENTARY-SWITCH-SPST-PTH-6.0MM" x="36.83" y="13.97" smashed="yes" rot="R180">
-<attribute name="PROD_ID" value=" SWCH-08441" x="36.83" y="13.97" size="1.778" layer="27" rot="R180" display="off"/>
-<attribute name="SF_SKU" value="COM-00097" x="36.83" y="13.97" size="1.778" layer="27" rot="R180" display="off"/>
-<attribute name="NAME" x="36.83" y="10.668" size="0.6096" layer="25" font="vector" ratio="20" rot="R180" align="bottom-center"/>
-</element>
-<element name="S5" library="SparkFun-Switches" package="TACTILE_SWITCH_PTH_6.0MM" value="MOMENTARY-SWITCH-SPST-PTH-6.0MM" x="57.15" y="13.97" smashed="yes" rot="R180">
-<attribute name="PROD_ID" value=" SWCH-08441" x="57.15" y="13.97" size="1.778" layer="27" rot="R180" display="off"/>
-<attribute name="SF_SKU" value="COM-00097" x="57.15" y="13.97" size="1.778" layer="27" rot="R180" display="off"/>
-<attribute name="NAME" x="57.15" y="10.668" size="0.6096" layer="25" font="vector" ratio="20" rot="R180" align="bottom-center"/>
-</element>
 <element name="U$3" library="Warthog9-Screens" package="OLED-I2C-4PIN" value="OLED-0.96I2C-4PIN" x="62.865" y="48.5775" smashed="yes">
 <attribute name="NAME" x="54.365" y="60.6775" size="0.6096" layer="25" font="vector" ratio="20"/>
@@
 <contactref element="S2" pad="1"/>
 <contactref element="S3" pad="1"/>
-<contactref element="S4" pad="1"/>
-<contactref element="S5" pad="1"/>
 <contactref element="U$3" pad="2"/>
 <contactref element="JP1" pad="3"/>
@@
 <contactref element="AMICA-NODEMCU" pad="D8"/>
 <contactref element="JP2" pad="14"/>
-<wire x1="100.33" y1="27.94" x2="100.33" y2="10.16" width="0" layer="19" extent="1-16"/>
 <wire x1="80.645" y1="72.0725" x2="80.645" y2="71.755" width="0.3048" layer="16"/>
 <wire x1="80.645" y1="71.755" x2="81.915" y2="70.485" width="0.3048" layer="16"/>
@@
 <via x="101.6" y="48.26" extent="1-16" drill="0.3048"/>
 <wire x1="101.6" y1="48.26" x2="101.6" y2="29.21" width="0.3048" layer="16"/>
-<wire x1="100.33" y1="27.94" x2="101.6" y2="29.21" width="0" layer="19" extent="1-16"/>
-<wire x1="52.7431" y1="10.16" x2="100.33" y2="10.16" width="0" layer="19" extent="1-16"/>
-<wire x1="100.33" y1="10.16" x2="100.33" y2="10.16" width="0" layer="19" extent="1-16"/>
 </signal>
 <signal name="GPIO0">
@@
 <signal name="GPIO10">
 <contactref element="AMICA-NODEMCU" pad="SD3"/>
-<contactref element="S5" pad="3"/>
 <contactref element="JP2" pad="6"/>
 <wire x1="70.485" y1="72.0725" x2="69.215" y2="70.8025" width="0.3048" layer="16"/>
@@
 <via x="83.82" y="16.1925" extent="1-16" drill="0.3048"/>
 <wire x1="83.82" y1="16.1925" x2="67.31" y2="16.1925" width="0.3048" layer="1"/>
-<wire x1="67.31" y1="16.1925" x2="60.4393" y2="16.1925" width="0.3048" layer="1"/>
-<wire x1="60.4393" y1="16.1925" x2="60.4012" y2="16.2306" width="0.3048" layer="1"/>
 <via x="67.31" y="16.1925" extent="1-16" drill="0.3048"/>
 <wire x1="67.31" y1="16.1925" x2="67.31" y2="31.75" width="0.3048" layer="16"/>
@@
 <signal name="GPIO9">
 <contactref element="AMICA-NODEMCU" pad="SD2"/>
-<contactref element="S4" pad="3"/>
 <contactref element="JP2" pad="19"/>
-<wire x1="86.36" y1="6.35" x2="86.36" y2="13.97" width="0.3048" layer="16"/>
-<wire x1="86.36" y1="13.97" x2="86.36" y2="25.4" width="0.3048" layer="16"/>
+<wire x1="86.36" y1="6.35" x2="86.36" y2="25.4" width="0.3048" layer="16"/>
 <wire x1="86.36" y1="25.4" x2="85.09" y2="26.67" width="0.3048" layer="16"/>
 <wire x1="85.09" y1="26.67" x2="85.09" y2="63.5" width="0.3048" layer="16"/>
 <wire x1="85.09" y1="63.5" x2="88.265" y2="66.675" width="0.3048" layer="16"/>
 <wire x1="88.265" y1="66.675" x2="88.265" y2="69.5325" width="0.3048" layer="16"/>
-<wire x1="40.0812" y1="16.2306" x2="40.0812" y2="15.7988" width="0.3048" layer="1"/>
-<wire x1="40.0812" y1="15.7988" x2="41.91" y2="13.97" width="0.3048" layer="1"/>
-<wire x1="41.91" y1="13.97" x2="86.36" y2="13.97" width="0.3048" layer="1"/>
-<via x="86.36" y="13.97" extent="1-16" drill="0.3048"/>
 </signal>
 <signal name="VCC">

Commit message: Removing GPIO9/10 from expansion header
These are unusable pins on enough NodeMCUs I'm going to go ahead
and remove the pins in the general sense
Connections:
- net GPIO10: no longer JP2.6
- net GPIO9: no longer JP2.19
Routing:
- net GPIO10: track 83.5 -> 0.00 mm, vias 2 -> 0
- net GPIO9: track 65.0 -> 0.00 mm
Other:
- board text removed: "IO10"
- board text removed: "IO9"
Changed lines of the file:
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@@
 <text x="65.405" y="73.3425" size="0.8128" layer="21" font="vector" rot="R45">TXD</text>
 <text x="67.945" y="73.3425" size="0.8128" layer="21" font="vector" rot="R45">RXD</text>
-<text x="70.485" y="73.3425" size="0.8128" layer="21" font="vector" rot="R45">IO10</text>
 <text x="73.025" y="73.3425" size="0.8128" layer="21" font="vector" rot="R45">IO12</text>
 <text x="75.565" y="73.3425" size="0.8128" layer="21" font="vector" rot="R45">IO13</text>
@@
 <text x="82.55" y="67.6275" size="0.8128" layer="21" font="vector" rot="R315">IO4</text>
 <text x="85.09" y="67.6275" size="0.8128" layer="21" font="vector" rot="R315">IO5</text>
-<text x="87.63" y="67.6275" size="0.8128" layer="21" font="vector" rot="R315">IO9</text>
 <text x="105.41" y="2.54" size="1.27" layer="22" font="vector" rot="MR0">https://github.com/warthog9/ABQMMF-Solderkit-2018</text>
 </plain>
@@
 <signal name="GPIO10">
 <contactref element="AMICA-NODEMCU" pad="SD3"/>
-<contactref element="JP2" pad="6"/>
-<wire x1="70.485" y1="72.0725" x2="69.215" y2="70.8025" width="0.3048" layer="16"/>
-<wire x1="83.82" y1="6.35" x2="83.82" y2="16.1925" width="0.3048" layer="16"/>
-<via x="83.82" y="16.1925" extent="1-16" drill="0.3048"/>
-<wire x1="83.82" y1="16.1925" x2="67.31" y2="16.1925" width="0.3048" layer="1"/>
-<via x="67.31" y="16.1925" extent="1-16" drill="0.3048"/>
-<wire x1="67.31" y1="16.1925" x2="67.31" y2="31.75" width="0.3048" layer="16"/>
-<wire x1="67.31" y1="31.75" x2="69.215" y2="33.655" width="0.3048" layer="16"/>
-<wire x1="69.215" y1="33.655" x2="69.215" y2="70.8025" width="0.3048" layer="16"/>
 </signal>
 <signal name="GPIO9">
 <contactref element="AMICA-NODEMCU" pad="SD2"/>
-<contactref element="JP2" pad="19"/>
-<wire x1="86.36" y1="6.35" x2="86.36" y2="25.4" width="0.3048" layer="16"/>
-<wire x1="86.36" y1="25.4" x2="85.09" y2="26.67" width="0.3048" layer="16"/>
-<wire x1="85.09" y1="26.67" x2="85.09" y2="63.5" width="0.3048" layer="16"/>
-<wire x1="85.09" y1="63.5" x2="88.265" y2="66.675" width="0.3048" layer="16"/>
-<wire x1="88.265" y1="66.675" x2="88.265" y2="69.5325" width="0.3048" layer="16"/>
 </signal>
 <signal name="VCC">

Commit message: Use the 0.96in OLED pinout that's got vcc/gnd reversed
Parts:
- U$3: value OLED-0.96I2C-4PIN -> OLED-0.96-VCCGND-REV; device Warthog9-Screens:OLED-I2C-4PIN -> Warthog9-Screens:OLED-I2C-4PIN-VCCGND-REV
Connections:
- net GND: now also U$3.1; no longer U$3.2
- net VCC: now also U$3.2; no longer U$3.1
Changed lines of the file:
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@@
 <attribute name="NAME" x="46.99" y="19.558" size="0.6096" layer="25" font="vector" ratio="20" rot="R180" align="bottom-center"/>
 </element>
-<element name="U$3" library="Warthog9-Screens" package="OLED-I2C-4PIN" value="OLED-0.96I2C-4PIN" x="62.865" y="48.5775" smashed="yes">
+<element name="U$3" library="Warthog9-Screens" package="OLED-I2C-4PIN-VCCGND-REV" value="OLED-0.96-VCCGND-REV" x="62.865" y="48.5775" smashed="yes">
 <attribute name="NAME" x="54.365" y="60.6775" size="0.6096" layer="25" font="vector" ratio="20"/>
 <attribute name="VALUE" x="69.18" y="52.5725" size="0.6096" layer="27" font="vector" ratio="20" rot="R90"/>
@@
 <contactref element="S2" pad="1"/>
 <contactref element="S3" pad="1"/>
-<contactref element="U$3" pad="2"/>
 <contactref element="JP1" pad="3"/>
 <contactref element="JP2" pad="3"/>
 <contactref element="JP2" pad="7"/>
+<contactref element="U$3" pad="1"/>
 </signal>
 <signal name="3.3V">
@@
 <contactref element="D1" pad="C"/>
 <contactref element="JP1" pad="4"/>
-<contactref element="U$3" pad="1"/>
 <contactref element="JP2" pad="1"/>
 <polygon width="0.3048" layer="16" rank="6">
@@
 <vertex x="0" y="95.25"/>
 </polygon>
+<contactref element="U$3" pad="2"/>
 </signal>
 <signal name="N$1">
